File: docs/electroCad/SteeringWheel.sch (KiCad schematic (older format))
At the start: 25 parts

Commit message: feat:split in moduls
Parts:
- SW301, SW302, SW303, SW304, SW305, SW306, SW307, SW308: renamed from SW?; footprint (none) -> Button_Switch_THT:SW_MEC_5GTH9
- gave numbers to parts that had none: 17
Connections:
- net at IOExt301.11 (P6): now also SW307.1, SW307.2
- no-connect marks 6 -> 12

Commit message: chore: add some info texts
Parts:
- renumbered ADC301 to ADC2, Display301 to Display0, IOExt301 to IOExt2, IOExt302 to IOExt3
Changed lines of the file:
@@
 P 2200 6000
 AR Path="/611115DA" Ref="ADC?"  Part="1"
-AR Path="/611353D7/611115DA" Ref="ADC301"  Part="1"
-F 0 "ADC301" H 2200 6681 50  0000 C CNN
+AR Path="/611353D7/611115DA" Ref="ADC2"  Part="1"
+F 0 "ADC2" H 2200 6681 50  0000 C CNN
 F 1 "ADS1115IDGS" H 2200 6590 50  0000 C CNN
 F 2 "Package_SO:TSSOP-10_3x3mm_P0.5mm" H 2200 5500 50  0001 C CNN
@@
 P 5050 5900
 AR Path="/61111607" Ref="Display?"  Part="1"
-AR Path="/611353D7/61111607" Ref="Display301"  Part="1"
-F 0 "Display301" H 5050 6681 50  0000 C CNN
+AR Path="/611353D7/61111607" Ref="Display0"  Part="1"
+F 0 "Display0" H 5050 6681 50  0000 C CNN
 F 1 "CR2013-MI2120" H 5050 6590 50  0000 C CNN
 F 2 "Display:CR2013-MI2120" H 5050 5200 50  0001 C CNN
@@
 P 2150 3600
 AR Path="/611116C1" Ref="IOExt?"  Part="1"
-AR Path="/611353D7/611116C1" Ref="IOExt302"  Part="1"
-F 0 "IOExt302" H 2150 4481 50  0000 C CNN
+AR Path="/611353D7/611116C1" Ref="IOExt3"  Part="1"
+F 0 "IOExt3" H 2150 4481 50  0000 C CNN
 F 1 "PCF8574" H 2150 4390 50  0000 C CNN
 F 2 "" H 2150 3600 50  0001 C CNN
@@
 P 2150 1500
 AR Path="/61111758" Ref="IOExt?"  Part="1"
-AR Path="/611353D7/61111758" Ref="IOExt301"  Part="1"
-F 0 "IOExt301" H 2150 2381 50  0000 C CNN
+AR Path="/611353D7/61111758" Ref="IOExt2"  Part="1"
+F 0 "IOExt2" H 2150 2381 50  0000 C CNN
 F 1 "PCF8574" H 2150 2290 50  0000 C CNN
 F 2 "" H 2150 1500 50  0001 C CNN
