File: docs/electroCad/ser4.sch (KiCad schematic (older format))
At the start: 27 parts, among them J1 DB15_Male, J2 DB15_Female_HighDensity, SW1 SW_MEC_5E, SW10 SW_MEC_5E, SW11 SW_MEC_5E, SW12 SW_MEC_5E, SW13 SW_MEC_5E, SW14 SW_MEC_5E, SW15 SW_MEC_5E, SW16 SW_MEC_5E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

Commit message: chore: split into multi sheets
Parts:
- removed ADC2: ADS1115IDGS, Package_SO:TSSOP-10_3x3mm_P0.5mm, symbol Analog_ADC:ADS1115IDGS
- removed Display0: CR2013-MI2120, Display:CR2013-MI2120, symbol Driver_Display:CR2013-MI2120
- removed IOExt2, IOExt3: PCF8574, symbol Interface_Expansion:PCF8574
- removed J1: DB15_Male, symbol Connector:DB15_Male
- removed J2: DB15_Female_HighDensity, symbol Connector:DB15_Female_HighDensity
- removed R-left1, R-right1: R-force, symbol Device:R_Variable_US
- removed R1, R2: 10k, symbol Device:R
- removed SW1, SW10, SW11, SW12, SW13, SW14, SW15, SW16, SW2, SW3, SW4, SW5, SW6, SW7, SW8, SW9: SW_MEC_5E, symbol Switch:SW_MEC_5E
- removed U3: ESP32-WROOM-32, RF_Module:ESP32-WROOM-32, symbol RF_Module:ESP32-WROOM-32
Connections:
- net labels removed: GND, VCC
- wire segments 186 -> 0
- no-connect marks 6 -> 0

Commit message: feat:split in moduls
Changed lines of the file:
@@
 $Descr A4 11693 8268
 encoding utf-8
-Sheet 1 3
+Sheet 1 4
 Title "SER4"
 Date "2021-08-07"
@@
 F1 "SteeringWheel.sch" 50
 $EndSheet
+$Sheet
+S 4900 950  3000 1400
+U 611C1B43
+F0 "Sheet611C1B42" 50
+F1 "SandBox.sch" 50
+$EndSheet
 $EndSCHEMATC

Commit message: chore: add some info texts
Other:
- note added: "Hinweise:\n- Das Huzzah32 ESP32 featherbord wird mit zwei parallelen Leisten gesteckt\n- Die WaveShare PCF8574 werden gesteckt (zwei 90° verdrehte Leisten mit 9 und 4 Pins)\n- Die Grove ADS1115 werden gesteckt (zwei 90° verdrehte Leisten mit 9 und 4 Pins)"
Changed lines of the file:
@@
 F1 "SandBox.sch" 50
 $EndSheet
+Text Notes 950  5800 0    50   ~ 0
+Hinweise:\n- Das Huzzah32 ESP32 featherbord wird mit zwei parallelen Leisten gesteckt\n- Die WaveShare PCF8574 werden gesteckt (zwei 90° verdrehte Leisten mit 9 und 4 Pins)\n- Die Grove ADS1115 werden gesteckt (zwei 90° verdrehte Leisten mit 9 und 4 Pins)
 $EndSCHEMATC
