File: docs/electroCad/ser4.kicad_pcb (KiCad board)
At the start: 2 copper layers, 159.8 x 99.8 mm, 0 parts

Commit message: feat:split in moduls
Parts:
- added ADC301: ADS1115IDGS, Package_SO:TSSOP-10_3x3mm_P0.5mm, F.Cu at (67.3, 101.8)
- added Display301: CR2013-MI2120, Display:CR2013-MI2120, F.Cu at (104.5, 84.0)
- added SW301: SW_MEC_5E, Button_Switch_THT:SW_MEC_5GTH9, F.Cu at (62.6, 53.6)
- added SW302: SW_MEC_5E, Button_Switch_THT:SW_MEC_5GTH9, F.Cu at (199.8, 53.6)
- added SW303: SW_MEC_5E, Button_Switch_THT:SW_MEC_5GTH9, F.Cu at (62.6, 71.3)
- added SW304: SW_MEC_5E, Button_Switch_THT:SW_MEC_5GTH9, F.Cu at (76.6, 66.3)
- added SW305: SW_MEC_5E, Button_Switch_THT:SW_MEC_5GTH9, F.Cu at (185.8, 66.3)
- added SW306: SW_MEC_5E, Button_Switch_THT:SW_MEC_5GTH9, F.Cu at (199.8, 71.3)
- added SW307: SW_MEC_5E, Button_Switch_THT:SW_MEC_5GTH9, F.Cu at (62.6, 129.8)
- added SW308: SW_MEC_5E, Button_Switch_THT:SW_MEC_5GTH9, F.Cu at (199.8, 129.8)

Commit message: chore: improve readme
Parts:
- removed ADC301: ADS1115IDGS, Package_SO:TSSOP-10_3x3mm_P0.5mm
- added ADC2: ADS1115IDGS, Package_SO:TSSOP-10_3x3mm_P0.5mm, F.Cu at (182.0, 92.9)
- renumbered Display301 to Display0
